Commit message: partially working

File: src/modular_arm_description/urdf/modular_arm.gazebo.xacro (robot description, xacro)
@@ -15,4 +15,5 @@
     </joint>
     <joint name="joint2">
+      <param name="initial_position">2.0</param>
       <command_interface name="position"/>
       <state_interface name="position"/>
@@ -20,4 +21,5 @@
     </joint>
     <joint name="joint3">
+      <param name="initial_position">-1.5</param>
       <command_interface name="position"/>
       <state_interface name="position"/>
@@ -25,4 +27,17 @@
     </joint>
     <joint name="joint4">
+      <param name="initial_position">-0.5</param>
+      <command_interface name="position"/>
+      <state_interface name="position"/>
+      <state_interface name="velocity"/>
+    </joint>
+    <joint name="finger_left_joint">
+      <param name="initial_position">0.0</param>
+      <command_interface name="position"/>
+      <state_interface name="position"/>
+      <state_interface name="velocity"/>
+    </joint>
+    <joint name="finger_right_joint">
+      <param name="initial_position">0.0</param>
       <command_interface name="position"/>
       <state_interface name="position"/>

File: src/modular_arm_description/urdf/modular_arm.urdf.xacro (robot description, xacro)
@@ -11,7 +11,14 @@
   <material name="orange"><color rgba="0.9 0.45 0.1 1.0"/></material>
   <material name="dark"><color rgba="0.2 0.2 0.2 1.0"/></material>
-  <!-- Reusable inertial block for a cylinder-ish link -->
-  <xacro:macro name="simple_inertial" params="mass">
+  <!-- Reusable inertial block. Uses a safe constant inertia (0.001) that
+       DART/ODE can handle numerically. Physically-exact inertias for small
+       links produce near-zero values (1e-7..1e-8) that overflow to NaN
+       during dynamics, crashing the ODE collision detector.
+       include_com: shift the COM to mid-link (z = length/2). -->
+  <xacro:macro name="simple_inertial" params="mass length include_com:=true">
     <inertial>
+      <xacro:if value="${include_com}">
+        <origin xyz="0 0 ${length/2}" rpy="0 0 0"/>
+      </xacro:if>
       <mass value="${mass}"/>
       <inertia ixx="0.001" ixy="0.0" ixz="0.0" iyy="0.001" iyz="0.0" izz="0.001"/>
@@ -31,5 +38,5 @@
         <geometry><cylinder radius="${link_radius}" length="${length}"/></geometry>
       </collision>
-      <xacro:simple_inertial mass="0.15"/>
+      <xacro:simple_inertial mass="0.15" length="${length}"/>
     </link>
   </xacro:macro>
@@ -48,5 +55,5 @@
       <geometry><cylinder radius="0.04" length="${L0}"/></geometry>
     </collision>
-    <xacro:simple_inertial mass="0.4"/>
+    <xacro:simple_inertial mass="0.4" length="${L0}"/>
   </link>
   <joint name="world_to_base" type="fixed">
@@ -66,5 +73,5 @@
       <geometry><sphere radius="0.025"/></geometry>
     </collision>
-    <xacro:simple_inertial mass="0.1"/>
+    <xacro:simple_inertial mass="0.1" length="0.0" include_com="false"/>
   </link>
   <joint name="joint1" type="revolute">
@@ -82,7 +89,7 @@
     <parent link="link1"/>
     <child link="link2"/>
-    <origin xyz="0 0 0" rpy="0 -1.5708 0"/>  <!-- link2's local +Z becomes world horizontal at theta2=0 -->
-    <axis xyz="0 1 0"/>
-    <limit lower="-1.5708" upper="1.5708" effort="${joint_effort}" velocity="${joint_velocity}"/>
+    <origin xyz="0 0 0" rpy="0 -1.5708 0"/>
+    <axis xyz="0 1 0"/>
+    <limit lower="-1.5708" upper="3.14159" effort="${joint_effort}" velocity="${joint_velocity}"/>
   </joint>
   <!-- =========================================================
@@ -95,5 +102,5 @@
     <origin xyz="0 0 ${L1}" rpy="0 0 0"/>
     <axis xyz="0 1 0"/>
-    <limit lower="-2.61799" upper="2.61799" effort="${joint_effort}" velocity="${joint_velocity}"/>
+    <limit lower="-3.14159" upper="3.14159" effort="${joint_effort}" velocity="${joint_velocity}"/>
   </joint>
   <!-- =========================================================
@@ -106,5 +113,5 @@
     <origin xyz="0 0 ${L2}" rpy="0 0 0"/>
     <axis xyz="0 1 0"/>
-    <limit lower="-2.0944" upper="2.0944" effort="${joint_effort}" velocity="${joint_velocity}"/>
+    <limit lower="-3.14159" upper="3.14159" effort="${joint_effort}" velocity="${joint_velocity}"/>
   </joint>
   <!-- =========================================================
@@ -117,4 +124,101 @@
     <origin xyz="0 0 ${L3}" rpy="0 0 0"/>
   </joint>
+  <!-- =========================================================
+       parallel-jaw gripper on the end effector
+       ========================================================= -->
+  <xacro:property name="gripper_spread" value="0.04"/>
+  <xacro:property name="finger_length" value="0.04"/>
+  <xacro:property name="finger_width" value="0.006"/>
+  <link name="gripper_base">
+    <visual>
+      <geometry><box size="0.025 0.05 0.015"/></geometry>
+      <material name="grey"/>
+    </visual>
+    <collision>
+      <geometry><box size="0.025 0.05 0.015"/></geometry>
+    </collision>
+    <xacro:simple_inertial mass="0.03" length="0.015" include_com="true"/>
+  </link>
+  <joint name="gripper_base_joint" type="fixed">
+    <parent link="end_effector_link"/>
+    <child link="gripper_base"/>
+    <origin xyz="0 0 0.006" rpy="0 0 0"/>
+  </joint>
+  <link name="finger_left">
+    <visual>
+      <origin xyz="0 0 ${finger_length/2}" rpy="0 0 0"/>
+      <geometry><box size="${finger_width} ${finger_width} ${finger_length}"/></geometry>
+      <material name="grey"/>
+    </visual>
+    <collision>
+      <origin xyz="0 0 ${finger_length/2}" rpy="0 0 0"/>
+      <geometry><box size="${finger_width} ${finger_width} ${finger_length}"/></geometry>
+    </collision>
+    <xacro:simple_inertial mass="0.005" length="0.0" include_com="false"/>
+  </link>
+  <joint name="finger_left_joint" type="prismatic">
+    <parent link="gripper_base"/>
+    <child link="finger_left"/>
+    <origin xyz="0 ${gripper_spread/2} 0.006" rpy="0 0 0"/>
+    <axis xyz="0 -1 0"/>
+    <limit lower="0" upper="${(gripper_spread - finger_width) / 2 - 0.001}" effort="1.0" velocity="0.1"/>
+  </joint>
+  <link name="finger_right">
+    <visual>
+      <origin xyz="0 0 ${finger_length/2}" rpy="0 0 0"/>
+      <geometry><box size="${finger_width} ${finger_width} ${finger_length}"/></geometry>
+      <material name="grey"/>
+    </visual>
+    <collision>
+      <origin xyz="0 0 ${finger_length/2}" rpy="0 0 0"/>
+      <geometry><box size="${finger_width} ${finger_width} ${finger_length}"/></geometry>
+    </collision>
+    <xacro:simple_inertial mass="0.005" length="0.0" include_com="false"/>
+  </link>
+  <joint name="finger_right_joint" type="prismatic">
+    <parent link="gripper_base"/>
+    <child link="finger_right"/>
+    <origin xyz="0 ${-gripper_spread/2} 0.006" rpy="0 0 0"/>
+    <axis xyz="0 1 0"/>
+    <limit lower="0" upper="${(gripper_spread - finger_width) / 2 - 0.001}" effort="1.0" velocity="0.1"/>
+  </joint>
+  <!-- =========================================================
+       wrist camera: mounted on gripper_base, looks forward at
+       the grasp zone — critical for LeRobot policy training
+       ========================================================= -->
+  <link name="wrist_camera_link">
+    <visual>
+      <geometry><box size="0.006 0.006 0.006"/></geometry>
+      <material name="grey"/>
+    </visual>
+    <collision>
+      <geometry><box size="0.006 0.006 0.006"/></geometry>
+    </collision>
+    <xacro:simple_inertial mass="0.001" length="0.0" include_com="false"/>
+  </link>
+  <joint name="wrist_camera_joint" type="fixed">
+    <parent link="gripper_base"/>
+    <child link="wrist_camera_link"/>
+    <origin xyz="0.012 0.0 0.008" rpy="0 1.5708 0"/>
+  </joint>
+  <gazebo reference="wrist_camera_link">
+    <sensor name="wrist_camera" type="camera">
+      <always_on>true</always_on>
+      <visualize>true</visualize>
+      <update_rate>30</update_rate>
+      <camera>
+        <horizontal_fov>1.0472</horizontal_fov>
+        <image>
+          <width>640</width>
+          <height>480</height>
+          <format>R8G8B8</format>
+        </image>
+        <clip>
+          <near>0.005</near>
+          <far>0.5</far>
+        </clip>
+      </camera>
+    </sensor>
+  </gazebo>
   <xacro:include filename="$(find modular_arm_description)/urdf/modular_arm.gazebo.xacro"/>
 </robot>
